Commit message: [mod] urdf mesh

File: humanSubjectWithSpinalCordMeshes/humanSubjectWithSpinalCordMeshes.urdf (robot description, URDF)
Before this commit: robot HumanModel, 103 links, 102 joints
Links:
- link Head: geometry collision sphere radius=0.108225; visual mesh filename=package://human-gazebo/humanSubjectWithSpinalCordMeshes/mes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 scale=1. 1. 1.
- link L3: geometry collision box size=0.06 0.1 0.074925; visual mesh filename=package://human-gazebo/humanSubjectWithSpinalCordMeshes/mes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 scale=1. 1. 1.
- link L5: geometry collision box size=0.06 0.1 0.0491175; visual mesh filename=package://human-gazebo/humanSubjectWithSpinalCordMeshes/mes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 scale=1. 1. 1.
- link LeftFoot: geometry collision box size=0.25308 0.091575 0.064935; visual mesh filename=package://human-gazebo/humanSubjectWithSpinalCordMeshes/mes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 scale=1. 1. 1.
- link LeftForeArm: geometry collision cylinder length=0.24309 radius=0.03503184713375795; visual mesh filename=package://human-gazebo/humanSubjectWithSpinalCordMeshes/mes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 scale=1. 1. 1.
- link LeftHand: geometry collision box size=0.085 0.17982 0.025; visual mesh filename=package://human-gazebo/humanSubjectWithSpinalCordMeshes/mes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 scale=1. 1. 1.
- link LeftHeel: geometry collision box size=0.0025308 0.091575 0.064935; visual mesh filename=package://human-gazebo/humanSubjectWithSpinalCordMeshes/mes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 scale=1. 1. 1.
- link LeftLowerLeg: geometry collision cylinder length=0.40959 radius=0.0541401274; visual mesh filename=package://human-gazebo/humanSubjectWithSpinalCordMeshes/mes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 scale=1. 1. 1.
- link LeftShoulder: geometry collision cylinder length=0.143745 radius=0.04617834395; visual mesh filename=package://human-gazebo/humanSubjectWithSpinalCordMeshes/mes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 scale=1. 1. 1.
- link LeftToe: geometry collision box size=0.0025308 0.091575 0.064935; visual mesh filename=package://human-gazebo/humanSubjectWithSpinalCordMeshes/mes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 scale=1. 1. 1.
- link LeftUpperArm: geometry collision cylinder length=0.30969 radius=0.04617834395; visual mesh filename=package://human-gazebo/humanSubjectWithSpinalCordMeshes/mes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 scale=1. 1. 1.
- link LeftUpperLeg: geometry collision cylinder length=0.407925 radius=0.0780254777; visual mesh filename=package://human-gazebo/humanSubjectWithSpinalCordMeshes/mes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 scale=1. 1. 1.
- link Neck: geometry collision cylinder length=0.08658 radius=0.05015923565; visual mesh filename=package://human-gazebo/humanSubjectWithSpinalCordMeshes/mes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 scale=1. 1. 1.
- link Pelvis: geometry collision box size=0.225 0.318015 0.12987; visual mesh filename=package://human-gazebo/humanSubjectWithSpinalCordMeshes/mes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 scale=1. 1. 1.
- link RightFoot: geometry collision box size=0.25308 0.091575 0.064935; visual mesh filename=package://human-gazebo/humanSubjectWithSpinalCordMeshes/mes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 scale=1. 1. 1.
- link RightForeArm: geometry collision cylinder length=0.24309 radius=0.03503184713375795; visual mesh filename=package://human-gazebo/humanSubjectWithSpinalCordMeshes/mes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 scale=1. 1. 1.
- link RightHand: geometry collision box size=0.085 0.17982 0.025; visual mesh filename=package://human-gazebo/humanSubjectWithSpinalCordMeshes/mes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 scale=1. 1. 1.
- link RightHeel: geometry collision box size=0.0025308 0.091575 0.064935; visual mesh filename=package://human-gazebo/humanSubjectWithSpinalCordMeshes/mes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 scale=1. 1. 1.
- link RightLowerLeg: geometry collision cylinder length=0.40959 radius=0.0541401274; visual mesh filename=package://human-gazebo/humanSubjectWithSpinalCordMeshes/mes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 scale=1. 1. 1.
- link RightShoulder: geometry collision cylinder length=0.143745 radius=0.04617834395; visual mesh filename=package://human-gazebo/humanSubjectWithSpinalCordMeshes/mes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 scale=1. 1. 1.
- link RightToe: geometry collision box size=0.0025308 0.091575 0.064935; visual mesh filename=package://human-gazebo/humanSubjectWithSpinalCordMeshes/mes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 scale=1. 1. 1.
- link RightUpperArm: geometry collision cylinder length=0.30969 radius=0.04617834395; visual mesh filename=package://human-gazebo/humanSubjectWithSpinalCordMeshes/mes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 scale=1. 1. 1.
- link RightUpperLeg: geometry collision cylinder length=0.407925 radius=0.0780254777; visual mesh filename=package://human-gazebo/humanSubjectWithSpinalCordMeshes/mes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 scale=1. 1. 1.
- link T12: geometry collision box size=0.06 0.1 0.087579; visual mesh filename=package://human-gazebo/humanSubjectWithSpinalCordMeshes/mes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 scale=1. 1. 1.
- link T8: geometry collision box size=0.06 0.143745 0.1380285; visual mesh filename=package://human-gazebo/humanSubjectWithSpinalCordMeshes/mes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 scale=1. 1. 1.
