Commit message: [mod] urdf mesh file path

File: humanSubjectWithMeshes/humanSubjectWithMesh.urdf (robot description, URDF)
Before this commit: robot HumanModel, 93 links, 92 joints
Links:
- link Head: geometry collision sphere radius=0.1105; visual mesh filename=package://human-gazebo/humanSubjectWithMeshes/meshes/Head.s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 scale=1.03030303 1.03030303 1.03030303
- link LeftFoot: geometry collision box size=0.2584 0.0935 0.0663; visual mesh filename=package://human-gazebo/humanSubjectWithMeshes/meshes/LeftFo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 scale=1.03030303 1.03030303 1.03030303
- link LeftForeArm: geometry collision cylinder length=0.24819999999999998 radius=0.0275; visual mesh filename=package://human-gazebo/humanSubjectWithMeshes/meshes/LeftEx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 scale=0.61111111 0.61111111 1.03030303
- link LeftHand: geometry collision box size=0.072 0.1836 0.025; visual mesh filename=package://human-gazebo/humanSubjectWithMeshes/meshes/LeftHa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 scale=0.9 1.03030303 0.55555556
- link LeftLowerLeg: geometry collision cylinder length=0.41819999999999996 radius=0.045; visual mesh filename=package://human-gazebo/humanSubjectWithMeshes/meshes/LeftGa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 scale=0.7826087 0.7826087 1.03030303
- link LeftShoulder: geometry collision cylinder length=0.14676666666666668 radius=0.029; visual mesh filename=package://human-gazebo/humanSubjectWithMeshes/meshes/LeftSh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 scale=0.64444444 0.64444444 1.03030303
- link LeftToe: geometry collision box size=0.002584 0.0935 0.0663; visual mesh filename=package://human-gazebo/humanSubjectWithMeshes/meshes/LeftTo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 scale=1.03030303 1.03030303 1.03030303
- link LeftUpperArm: geometry collision cylinder length=0.3162 radius=0.029; visual mesh filename=package://human-gazebo/humanSubjectWithMeshes/meshes/LeftBi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 scale=0.64444444 0.64444444 1.03030303
- link LeftUpperLeg: geometry collision cylinder length=0.4165 radius=0.0625; visual mesh filename=package://human-gazebo/humanSubjectWithMeshes/meshes/LeftBi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 scale=0.83333333 0.83333333 1.03030303
- link LowerTrunk: geometry collision box size=0.175 0.2958 0.17; visual mesh filename=package://human-gazebo/humanSubjectWithMeshes/meshes/LowerT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 scale=0.58333333 1.03030303 1.03030303
- link Neck: geometry collision cylinder length=0.08839999999999999 radius=0.0475; visual mesh filename=package://human-gazebo/humanSubjectWithMeshes/meshes/Neck.s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 scale=0.73076923 0.73076923 1.03030303
- link Pelvis: geometry collision box size=0.175 0.3247 0.1326; visual mesh filename=package://human-gazebo/humanSubjectWithMeshes/meshes/Pelvis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 scale=0.58333333 1.03030303 1.03030303
- link RightFoot: geometry collision box size=0.2584 0.0935 0.0663; visual mesh filename=package://human-gazebo/humanSubjectWithMeshes/meshes/RightF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 scale=1.03030303 1.03030303 1.03030303
- link RightForeArm: geometry collision cylinder length=0.24819999999999998 radius=0.0275; visual mesh filename=package://human-gazebo/humanSubjectWithMeshes/meshes/RightE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 scale=0.61111111 0.61111111 1.03030303
- link RightHand: geometry collision box size=0.072 0.1836 0.025; visual mesh filename=package://human-gazebo/humanSubjectWithMeshes/meshes/RightH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 scale=0.9 1.03030303 0.55555556
- link RightLowerLeg: geometry collision cylinder length=0.41819999999999996 radius=0.045; visual mesh filename=package://human-gazebo/humanSubjectWithMeshes/meshes/RightG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 scale=0.7826087 0.7826087 1.03030303
- link RightShoulder: geometry collision cylinder length=0.14676666666666668 radius=0.029; visual mesh filename=package://human-gazebo/humanSubjectWithMeshes/meshes/RightS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 scale=0.64444444 0.64444444 1.03030303
- link RightToe: geometry collision box size=0.002584 0.0935 0.0663; visual mesh filename=package://human-gazebo/humanSubjectWithMeshes/meshes/RightT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 scale=1.03030303 1.03030303 1.03030303
- link RightUpperArm: geometry collision cylinder length=0.3162 radius=0.029; visual mesh filename=package://human-gazebo/humanSubjectWithMeshes/meshes/RightB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 scale=0.64444444 0.64444444 1.03030303
- link RightUpperLeg: geometry collision cylinder length=0.4165 radius=0.0625; visual mesh filename=package://human-gazebo/humanSubjectWithMeshes/meshes/RightB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 scale=0.83333333 0.83333333 1.03030303
- link UpperTrunk: geometry collision box size=0.175 0.14676667 0.187; visual mesh filename=package://human-gazebo/humanSubjectWithMeshes/meshes/UpperT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 scale=0.58333333 1.03030303 1.03030303

Commit message: [add] contact without testing

File: humanSubjectWithMeshes/humanSubjectWithMesh.urdf (robot description, URDF)
Before this commit: robot HumanModel, 93 links, 92 joints
Links:
- added link left_contact, mass 0.001; visual box size=0 0 0
- added link right_contact, mass 0.001; visual box size=0 0 0
Joints:
- added joint left_contact_fix: type fixed, parent LeftFoot, child left_contact, origin xyz=0 0.047 0 rpy=1.5707963267948966 0 0
- added joint right_contact_fix: type fixed, parent RightFoot, child right_contact, origin xyz=0 0.047 0 rpy=1.5707963267948966 0 0

Commit message: [mod] change Pelvis to base

File: humanSubjectWithMeshes/humanSubjectWithMesh.urdf (robot description, URDF)
Before this commit: robot HumanModel, 95 links, 94 joints
Links:
- removed link Pelvis
- added link base, mass 7.098; collision box size=0.175 0.3247 0.1326; visual mesh filename=package://human-gazebo/humanSubjectWithMeshes/meshes/Pelvis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 scale=0.58333333 1.03030303 1.03030303
Joints:
- joint jL5S1_rotx: parent Pelvis -> base
- joint jLeftErSpin_LP: parent Pelvis -> base
- joint jLeftHip_rotx: parent Pelvis -> base
- joint jLeftRecAbd_LP: parent Pelvis -> base
- joint jLeftRecFem_LP: parent Pelvis -> base
- joint jRightErSpin_RP: parent Pelvis -> base
- joint jRightHip_rotx: parent Pelvis -> base
- joint jRightRecAbd_RP: parent Pelvis -> base
- joint jRightRecFem_RP: parent Pelvis -> base

Commit message: [mod] minor modify link position

File: humanSubjectWithMeshes/humanSubjectWithMesh.urdf (robot description, URDF)
Before this commit: robot HumanModel, 95 links, 94 joints
Joints:
- joint left_contact_fix: origin xyz=0 0.047 0 rpy=1.5707963267948966 0 0 -> xyz=0 0 0 rpy=1.5707963267948966 0 0
- joint right_contact_fix: origin xyz=0 0.047 0 rpy=1.5707963267948966 0 0 -> xyz=0 0 0 rpy=1.5707963267948966 0 0

Commit message: [mod] modify joint names & modify toe angle limit

File: humanSubjectWithMeshes/humanSubjectWithMesh.urdf (robot description, URDF)
Before this commit: robot HumanModel, 95 links, 94 joints
Joints:
- removed joint jC1Head_rotx
- removed joint jC1Head_roty
- removed joint jC7LeftShoulder_rotx
- removed joint jC7RightShoulder_rotx
- removed joint jL5S1_rotx
- removed joint jL5S1_roty
- removed joint jLeftBallFoot_roty
- removed joint jRightBallFoot_roty
- removed joint jT1C7_rotx
- removed joint jT1C7_roty
- removed joint jT1C7_rotz
- removed joint jT9T8_rotx
- removed joint jT9T8_roty
- removed joint jT9T8_rotz
- added joint jHead_rotx: type revolute, parent Neck, child Head_f1, origin xyz=0.0 0.0 0.08839999999999999 rpy=0.0 0.0 0.0, axis 1. 0. 0., limit lower=-0.610865 upper=0.610865 effort=30.0 velocity=1.0
- added joint jHead_roty: type revolute, parent Head_f1, child Head, origin xyz=0.0 0.0 0.0 rpy=0.0 0.0 0.0, axis 0. 1. 0., limit lower=-0.436332 upper=0.174533 effort=30.0 velocity=1.0
- added joint jLeftToe_roty: type revolute, parent LeftFoot, child LeftToe, origin xyz=0.21469199999999997 0.0 -0.03315 rpy=0.0 0.0 0.0, axis 0. 1. 0., limit lower=2.967057 upper=3.316122 effort=30.0 velocity=1.0
- added joint jNeck_rotx: type revolute, parent UpperTrunk, child Neck_f1, origin xyz=0.0 0.0 0.187 rpy=0.0 0.0 0.0, axis 1. 0. 0., limit lower=-0.610865 upper=0.610865 effort=30.0 velocity=1.0
- added joint jNeck_roty: type revolute, parent Neck_f1, child Neck_f2, origin xyz=0.0 0.0 0.0 rpy=0.0 0.0 0.0, axis 0. 1. 0., limit lower=-0.959931 upper=1.5708 effort=30.0 velocity=1.0
- added joint jNeck_rotz: type revolute, parent Neck_f2, child Neck, origin xyz=0.0 0.0 0.0 rpy=0.0 0.0 0.0, axis 0. 0. 1., limit lower=-1.22173 upper=1.22173 effort=30.0 velocity=1.0
- added joint jRightToe_roty: type revolute, parent RightFoot, child RightToe, origin xyz=0.21469199999999997 0.0 -0.03315 rpy=0.0 0.0 0.0, axis 0. 1. 0., limit lower=2.967057 upper=3.316122 effort=30.0 velocity=1.0
- added joint jSpineChest_rotx: type revolute, parent LowerTrunk, child UpperTrunk_f1, origin xyz=0.0 0.0 0.17 rpy=0.0 0.0 0.0, axis 1. 0. 0., limit lower=-0.349066 upper=0.349066 effort=30.0 velocity=1.0
- added joint jSpineChest_roty: type revolute, parent UpperTrunk_f1, child UpperTrunk_f2, origin xyz=0.0 0.0 0.0 rpy=0.0 0.0 0.0, axis 0. 1. 0., limit lower=-0.261799 upper=0.698132 effort=30.0 velocity=1.0
- added joint jSpineChest_rotz: type revolute, parent UpperTrunk_f2, child UpperTrunk, origin xyz=0.0 0.0 0.0 rpy=0.0 0.0 0.0, axis 0. 0. 1., limit lower=-0.610865 upper=0.610865 effort=30.0 velocity=1.0
- added joint jSpineNaval_rotx: type revolute, parent base, child LowerTrunk_f1, origin xyz=0.0 0.0 0.0663 rpy=0.0 0.0 0.0, axis 1. 0. 0., limit lower=-0.610865 upper=0.610865 effort=30.0 velocity=1.0
- added joint jSpineNaval_roty: type revolute, parent LowerTrunk_f1, child LowerTrunk, origin xyz=0.0 0.0 0.0 rpy=0.0 0.0 0.0, axis 0. 1. 0., limit lower=-0.523599 upper=1.309 effort=30.0 velocity=1.0

Commit message: [fix] change Shoulder to Clavicle

File: humanSubjectWithMeshes/humanSubjectWithMesh.urdf (robot description, URDF)
Before this commit: robot HumanModel, 95 links, 92 joints
Joints:
- added joint jLeftClavicleShoulder_rotx: type revolute, parent UpperTrunk, child LeftShoulder, origin xyz=0.0 0.07338333333333334 0.158 rpy=0.0 0.0 0.0, axis 1. 0. 0., limit lower=-0.0872665 upper=0.785398 effort=30.0 velocity=1.0
- added joint jRightClavicleShoulder_rotx: type revolute, parent UpperTrunk, child RightShoulder, origin xyz=0.0 -0.07338333333333334 0.158 rpy=0.0 0.0 0.0, axis 1. 0. 0., limit lower=-0.785398 upper=0.0872665 effort=30.0 velocity=1.0

Commit message: [mod] change Toe back to original limit

File: humanSubjectWithMeshes/humanSubjectWithMesh.urdf (robot description, URDF)
Before this commit: robot HumanModel, 95 links, 94 joints
Joints:
- joint jLeftToe_roty: limit lower=2.967057 upper=3.316122 effort=30.0 velocity=1.0 -> lower=-0.174533 upper=1.5708 effort=30.0 velocity=1.0
- joint jRightToe_roty: limit lower=2.967057 upper=3.316122 effort=30.0 velocity=1.0 -> lower=-0.174533 upper=1.5708 effort=30.0 velocity=1.0
